File: hardware/notchdeck-one/notchdeck-one.kicad_sch (KiCad schematic)
At the start: 0 parts

Commit message: Add schgen schematic workflow + flatten extends symbols
Brings notchdeck onto the data-manifest schematic workflow (scripts/kschgen.py
+ notchdeck-one.schgen.py, Makefile gen/check/render targets, project skills,
CLAUDE.md) and commits the generated hierarchical child sheets (mcu/power/
lever/controls), which were previously untracked.

kschgen fix: flatten extends-based symbols. kicad-cli's SVG/PDF exporters don't
resolve (extends ...), so derived symbols (e.g. the TC2030-NL SWD connector)
rendered blank. _flattened_block() now inlines the parent's graphics/pins,
renamed to the child, dropping the extends — so generated sheets render
correctly outside eeschema. (Same fix landed in ephemerkey.)

make check-notchdeck-one: 74 components, 74/74 footprints, no dup refs.

Co-Authored-By: Claude Opus 4.8 (1M context) <noreply@anthropic.com>
Other:
- added sheet Controls (controls.kicad_sch)
- added sheet Lever (lever.kicad_sch)
- added sheet MCU (mcu.kicad_sch)
- added sheet Power (power.kicad_sch)
Changed lines of the file:
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@@
 		(company "BenchBits")
 		(comment 1 "Dual-mode (USB + BLE) one-handle train master controller")
-		(comment 2 "Empty scaffold — populate per hardware/PARTS.md")
+		(comment 2 "Top-level — hierarchical sheets per functional block")
+	)
+	(sheet
+		(at 40.64 40.64)
+		(size 36.00 22.00)
+		(fields_autoplaced yes)
+		(stroke (width 0.1524) (type solid))
+		(fill (color 0 0 0 0.0000))
+		(property "Sheetname" "MCU"
+			(at 40.64 39.37 0)
+			(effects (font (size 1.27 1.27)) (justify left bottom))
+		)
+		(property "Sheetfile" "mcu.kicad_sch"
+			(at 40.64 63.91 0)
+			(effects (font (size 1.27 1.27)) (justify left top))
+		)
+	)
+	(sheet
+		(at 96.52 40.64)
+		(size 36.00 22.00)
+		(fields_autoplaced yes)
+		(stroke (width 0.1524) (type solid))
+		(fill (color 0 0 0 0.0000))
+		(property "Sheetname" "Power"
+			(at 96.52 39.37 0)
+			(effects (font (size 1.27 1.27)) (justify left bottom))
+		)
+		(property "Sheetfile" "power.kicad_sch"
+			(at 96.52 63.91 0)
+			(effects (font (size 1.27 1.27)) (justify left top))
+		)
+	)
+	(sheet
+		(at 152.40 40.64)
+		(size 36.00 22.00)
+		(fields_autoplaced yes)
+		(stroke (width 0.1524) (type solid))
+		(fill (color 0 0 0 0.0000))
+		(property "Sheetname" "Lever"
+			(at 152.40 39.37 0)
+			(effects (font (size 1.27 1.27)) (justify left bottom))
+		)
+		(property "Sheetfile" "lever.kicad_sch"
+			(at 152.40 63.91 0)
+			(effects (font (size 1.27 1.27)) (justify left top))
+		)
+	)
+	(sheet
+		(at 208.28 40.64)
+		(size 36.00 22.00)
+		(fields_autoplaced yes)
+		(stroke (width 0.1524) (type solid))
+		(fill (color 0 0 0 0.0000))
+		(property "Sheetname" "Controls"
+			(at 208.28 39.37 0)
+			(effects (font (size 1.27 1.27)) (justify left bottom))
+		)
+		(property "Sheetfile" "controls.kicad_sch"
+			(at 208.28 63.91 0)
+			(effects (font (size 1.27 1.27)) (justify left top))
+		)
 	)
 	(sheet_instances
