File: hardware/notchdeck-one/mcu.kicad_sch (KiCad schematic)
At the start: 10 parts, among them J3 SWD, J4 TC2030_NL, SW17 RESET, U1 E73-2G4M08S1C

Commit message: Split controller buttons onto stocked STM32G030 panel PCB
Connections:
- net BTN1 renamed PANEL_INT
- net BTN10: no longer names the net of U1.43 (P0.10/NFC2)
- net BTN11: no longer names the net of U1.11 (P0.00/XL1)
- net BTN12: no longer names the net of U1.13 (P0.01/XL2)
- net BTN2: no longer names the net of U1.2 (P1.10)
- net BTN3: no longer names the net of U1.6 (P1.13)
- net BTN4: no longer names the net of U1.17 (P1.09)
- net BTN5: no longer names the net of U1.32 (P0.20)
- net BTN6: no longer names the net of U1.33 (P0.13)
- net BTN9: no longer names the net of U1.41 (P0.09/NFC1)
- net HAT_DOWN: no longer names the net of U1.35 (P0.24)
- net HAT_LEFT: no longer names the net of U1.36 (P1.00)
- net HAT_RIGHT: no longer names the net of U1.38 (P1.02)
- net HAT_UP: no longer names the net of U1.34 (P0.22)
- net WS2812_DIN: no longer names the net of U1.16 (P0.08)
- no-connect marks 5 -> 19
Other:
- note added: "SWD headers are parallel; VTref is 3V3. SWO is unused. Reset: P0.18 / UICR reset enabled; also resets handle mux. Rev E leaves NFC pins unconnected; no NFC pin setup required. Rev E frees 14 GPIOs; still use calibrated RC LFCLK, no LFXO. P0.29/P0.31/P0.30 = power Gray bits S0/S1/S2. P1.11 = panel IRQ."
- note removed: "SWD headers are parallel; VTref is 3V3. SWO is unused. Reset: P0.18 / UICR reset enabled; also resets handle mux. NFC pins P0.09/P0.10 must be configured as GPIO. P0.00/P0.01 are buttons: use calibrated RC LFCLK, no LFXO. P0.29/P0.31/P0.30 = power Gray bits S0/S1/S2. No spare GPIO."

Commit message: Add protected PWM actuator outputs and charger interlock
Connections:
- net SOL1_PWM: now reaches U1.32 (P0.20)
- net SOL2_PWM: now reaches U1.33 (P0.13)
- net BUZZ_PWM: now reaches U1.34 (P0.22)
- net ACT_EN: now reaches U1.35 (P0.24)
- net ACT_nFAULT: now reaches U1.36 (P1.00)
- no-connect marks 19 -> 14
Other:
- note added: "SWD headers are parallel; VTref is 3V3. SWO is unused. Reset: P0.18 / UICR reset enabled; also resets handle mux. Rev F: P0.20 SOL1, P0.13 SOL2, P0.22 BUZZ; active high. 9 spare GPIOs; calibrated RC LFCLK, no LFXO/NFC. Actuator firmware must default OFF; see ACTUATORS.md."
- note removed: "SWD headers are parallel; VTref is 3V3. SWO is unused. Reset: P0.18 / UICR reset enabled; also resets handle mux. Rev E leaves NFC pins unconnected; no NFC pin setup required. Rev E frees 14 GPIOs; still use calibrated RC LFCLK, no LFXO. P0.29/P0.31/P0.30 = power Gray bits S0/S1/S2. P1.11 = panel IRQ."
Changed lines of the file:
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@@
 	(title_block
 		(title "NotchDeck One — MCU & Programming")
-		(date "2026-10-03")
-		(rev "E")
+		(date "2026-10-04")
+		(rev "F")
 		(company "BenchBits")
 	)
@@
 		(stroke (width 0) (type default))
 	)
+	(wire (pts (xy 118.1100 68.5800) (xy 123.1900 68.5800))
+		(stroke (width 0) (type default))
+	)
+	(wire (pts (xy 118.1100 71.1200) (xy 123.1900 71.1200))
+		(stroke (width 0) (type default))
+	)
+	(wire (pts (xy 118.1100 73.6600) (xy 123.1900 73.6600))
+		(stroke (width 0) (type default))
+	)
+	(wire (pts (xy 118.1100 76.2000) (xy 123.1900 76.2000))
+		(stroke (width 0) (type default))
+	)
+	(wire (pts (xy 118.1100 78.7400) (xy 123.1900 78.7400))
+		(stroke (width 0) (type default))
+	)
 	(wire (pts (xy 118.1100 81.2800) (xy 123.1900 81.2800))
 		(stroke (width 0) (type default))
@@
 	)
 	(wire (pts (xy 335.2800 152.4000) (xy 360.6800 152.4000))
+		(stroke (width 0) (type default))
+	)
+	(wire (pts (xy 335.2800 158.7500) (xy 360.6800 158.7500))
+		(stroke (width 0) (type default))
+	)
+	(wire (pts (xy 335.2800 165.1000) (xy 360.6800 165.1000))
+		(stroke (width 0) (type default))
+	)
+	(wire (pts (xy 335.2800 171.4500) (xy 360.6800 171.4500))
+		(stroke (width 0) (type default))
+	)
+	(wire (pts (xy 335.2800 177.8000) (xy 360.6800 177.8000))
+		(stroke (width 0) (type default))
+	)
+	(wire (pts (xy 335.2800 184.1500) (xy 360.6800 184.1500))
 		(stroke (width 0) (type default))
 	)
@@
 	(label "USB_DP"
 		(at 123.1900 81.2800 0)
+		(effects (font (size 1.27 1.27)) (justify left bottom))
+	)
+	(label "SOL1_PWM"
+		(at 123.1900 78.7400 0)
+		(effects (font (size 1.27 1.27)) (justify left bottom))
+	)
+	(label "SOL2_PWM"
+		(at 123.1900 76.2000 0)
+		(effects (font (size 1.27 1.27)) (justify left bottom))
+	)
+	(label "BUZZ_PWM"
+		(at 123.1900 73.6600 0)
+		(effects (font (size 1.27 1.27)) (justify left bottom))
+	)
+	(label "ACT_EN"
+		(at 123.1900 71.1200 0)
+		(effects (font (size 1.27 1.27)) (justify left bottom))
+	)
+	(label "ACT_nFAULT"
+		(at 123.1900 68.5800 0)
 		(effects (font (size 1.27 1.27)) (justify left bottom))
 	)
@@
 	(no_connect (at 83.82 86.36))
 	(no_connect (at 83.82 88.9))
-	(no_connect (at 118.11 78.74))
-	(no_connect (at 118.11 76.2))
-	(no_connect (at 118.11 73.66))
-	(no_connect (at 118.11 71.12))
-	(no_connect (at 118.11 68.58))
 	(no_connect (at 118.11 63.5))
 	(no_connect (at 118.11 55.88))
@@
 		(effects (font (size 1.27 1.27)) (justify left bottom))
 	)
+	(hierarchical_label "SOL1_PWM"
+		(shape bidirectional)
+		(at 335.2800 158.7500 180)
+		(effects (font (size 1.27 1.27)) (justify right))
+	)
+	(label "SOL1_PWM"
+		(at 360.6800 158.7500 0)
+		(effects (font (size 1.27 1.27)) (justify left bottom))
+	)
+	(hierarchical_label "SOL2_PWM"
+		(shape bidirectional)
+		(at 335.2800 165.1000 180)
+		(effects (font (size 1.27 1.27)) (justify right))
+	)
+	(label "SOL2_PWM"
+		(at 360.6800 165.1000 0)
+		(effects (font (size 1.27 1.27)) (justify left bottom))
+	)
+	(hierarchical_label "BUZZ_PWM"
+		(shape bidirectional)
+		(at 335.2800 171.4500 180)
+		(effects (font (size 1.27 1.27)) (justify right))
+	)
+	(label "BUZZ_PWM"
+		(at 360.6800 171.4500 0)
+		(effects (font (size 1.27 1.27)) (justify left bottom))
+	)
+	(hierarchical_label "ACT_EN"
+		(shape bidirectional)
+		(at 335.2800 177.8000 180)
+		(effects (font (size 1.27 1.27)) (justify right))
+	)
+	(label "ACT_EN"
+		(at 360.6800 177.8000 0)
+		(effects (font (size 1.27 1.27)) (justify left bottom))
+	)
+	(hierarchical_label "ACT_nFAULT"
+		(shape bidirectional)
+		(at 335.2800 184.1500 180)
+		(effects (font (size 1.27 1.27)) (justify right))
+	)
+	(label "ACT_nFAULT"
+		(at 360.6800 184.1500 0)
+		(effects (font (size 1.27 1.27)) (justify left bottom))
+	)
 	(text "3V3 decoupling: C1/C3 at VDD; C2/C4 at VDDH.\nC5 bulk. VDD = VDDH; DCCH intentionally open."
 		(exclude_from_sim no)
@@
 		(effects (font (face "Courier New") (size 1.27 1.27)) (justify left top))
 	)
-	(text "SWD headers are parallel; VTref is 3V3. SWO is unused.\nReset: P0.18 / UICR reset enabled; also resets handle mux.\nRev E leaves NFC pins unconnected; no NFC pin setup required.\nRev E frees 14 GPIOs; still use calibrated RC LFCLK, no LFXO.\nP0.29/P0.31/P0.30 = power Gray bits S0/S1/S2. P1.11 = panel IRQ."
+	(text "SWD headers are parallel; VTref is 3V3. SWO is unused.\nReset: P0.18 / UICR reset enabled; also resets handle mux.\nRev F: P0.20 SOL1, P0.13 SOL2, P0.22 BUZZ; active high.\n9 spare GPIOs; calibrated RC LFCLK, no LFXO/NFC.\nActuator firmware must default OFF; see ACTUATORS.md."
 		(exclude_from_sim no)
 		(at 25.40 223.52 0)

Commit message: Protect full battery input and size dual 2A impulse outputs
Connections:
- net ACT_nFAULT renamed BAT_nFAULT
Other:
- note added: "SWD headers are parallel; VTref is 3V3. SWO is unused. Reset: P0.18 / UICR reset enabled; also resets handle mux. Rev G: P0.20 SOL1, P0.13 SOL2, P0.22 BUZZ; active high. 9 spare GPIOs; calibrated RC LFCLK, no LFXO/NFC. Actuator firmware must default OFF; see ACTUATORS.md."
- note removed: "SWD headers are parallel; VTref is 3V3. SWO is unused. Reset: P0.18 / UICR reset enabled; also resets handle mux. Rev F: P0.20 SOL1, P0.13 SOL2, P0.22 BUZZ; active high. 9 spare GPIOs; calibrated RC LFCLK, no LFXO/NFC. Actuator firmware must default OFF; see ACTUATORS.md."
Changed lines of the file:
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@@
 		(title "NotchDeck One — MCU & Programming")
 		(date "2026-10-04")
-		(rev "F")
+		(rev "G")
 		(company "BenchBits")
 	)
@@
 		(effects (font (size 1.27 1.27)) (justify left bottom))
 	)
-	(label "ACT_nFAULT"
+	(label "BAT_nFAULT"
 		(at 123.1900 68.5800 0)
 		(effects (font (size 1.27 1.27)) (justify left bottom))
@@
 		(effects (font (size 1.27 1.27)) (justify left bottom))
 	)
-	(hierarchical_label "ACT_nFAULT"
+	(hierarchical_label "BAT_nFAULT"
 		(shape bidirectional)
 		(at 335.2800 184.1500 180)
 		(effects (font (size 1.27 1.27)) (justify right))
 	)
-	(label "ACT_nFAULT"
+	(label "BAT_nFAULT"
 		(at 360.6800 184.1500 0)
 		(effects (font (size 1.27 1.27)) (justify left bottom))
@@
 		(effects (font (face "Courier New") (size 1.27 1.27)) (justify left top))
 	)
-	(text "SWD headers are parallel; VTref is 3V3. SWO is unused.\nReset: P0.18 / UICR reset enabled; also resets handle mux.\nRev F: P0.20 SOL1, P0.13 SOL2, P0.22 BUZZ; active high.\n9 spare GPIOs; calibrated RC LFCLK, no LFXO/NFC.\nActuator firmware must default OFF; see ACTUATORS.md."
+	(text "SWD headers are parallel; VTref is 3V3. SWO is unused.\nReset: P0.18 / UICR reset enabled; also resets handle mux.\nRev G: P0.20 SOL1, P0.13 SOL2, P0.22 BUZZ; active high.\n9 spare GPIOs; calibrated RC LFCLK, no LFXO/NFC.\nActuator firmware must default OFF; see ACTUATORS.md."
 		(exclude_from_sim no)
 		(at 25.40 223.52 0)
